Commit message: vision: fixing nan problem semantic_mapping: fixes in object mapping prob_map_viewer: added object location window launch files for rtabmap

File: hardware/urdf/sensors/own_sensors.urdf.xacro (robot description, xacro)
@@ -11,5 +11,5 @@
   <xacro:macro name="own_sensors" params="parent">
     <joint name="camera_joint" type="fixed">
-      <origin xyz="-0.1 0.0 1.03"
+      <origin xyz="-0.15 0.0 1.03"
               rpy="0.01 0.2 -0.02"/>
       <parent link="${parent}"/>

Commit message: better settings for camera transformation

File: hardware/urdf/sensors/own_sensors.urdf.xacro (robot description, xacro)
@@ -11,6 +11,6 @@
   <xacro:macro name="own_sensors" params="parent">
     <joint name="camera_joint" type="fixed">
-      <origin xyz="-0.15 0.0 1.03"
-              rpy="0.01 0.2 -0.02"/>
+      <origin xyz="-0.18 0.0 0.98"
+              rpy="-0.025 0.17 -0.008"/>
       <parent link="${parent}"/>
       <child link="camera_link" />

Commit message: setting up mapping package with everything included vision changed to gaussian representation of object location multi_asus in launchfiles

File: hardware/urdf/sensors/own_sensors.urdf.xacro (robot description, xacro)
@@ -10,4 +10,5 @@
   <!-- Parameterised in part by the values in turtlebot_properties.urdf.xacro -->
   <xacro:macro name="own_sensors" params="parent">
+    <!-- Main Asus -->
     <joint name="camera_joint" type="fixed">
       <origin xyz="-0.18 0.0 0.98"
@@ -112,4 +113,84 @@
       </inertial>
     </link>
+    <!-- Door detection Asus -->
+    <joint name="door_asus/camera_joint" type="fixed">
+      <origin xyz="-0.18 -0.03 0.65"
+              rpy="-0.035 -1.13 0.07"/>
+      <parent link="${parent}"/>
+      <child link="door_asus/camera_link" />
+    </joint>
+    <link name="door_asus/camera_link">
+      <visual>
+        <origin xyz="-0.015 0.0035 0.004" rpy="0 0 0"/>
+        <geometry>
+          <mesh filename="package://turtlebot_description/meshes/sensors/xtion_pro_camera.dae"/>
+        </geometry>
+      </visual>
+      <collision>
+        <origin xyz="0.0 0.0 0.0" rpy="0 0 0" />
+        <geometry>
+        <box size="0.0730 0.2760 0.0720"/>
+      </geometry>
+      </collision>
+      <inertial>
+        <mass value="0.170" />
+        <origin xyz="0 0 0" />
+        <inertia ixx="0.001152600" ixy="0.0" ixz="0.0"
+                 iyy="0.000148934" iyz="0.0"
+                 izz="0.001154654" />
+      </inertial>
+    </link>
+    <joint name="door_asus/camera_rgb_optical_joint" type="fixed">
+      <origin xyz="0 0 0" rpy="${-M_PI/2} 0 ${-M_PI/2}" />
+      <parent link="door_asus/camera_rgb_frame" />
+      <child link="door_asus/camera_rgb_optical_frame" />
+    </joint>
+    <link name="door_asus/camera_rgb_optical_frame"/>
+    <joint name="door_asus/camera_rgb_joint" type="fixed">
+      <origin xyz="0 ${asus_xtion_pro_cam_rel_rgb_py} 0"
+              rpy="0 0 0"/>
+      <parent link="door_asus/camera_link"/>
+      <child link="door_asus/camera_rgb_frame"/>
+    </joint>
+    <link name="door_asus/camera_rgb_frame"/>
+    <joint name="door_asus/camera_depth_joint" type="fixed">
+      <origin xyz="0 ${asus_xtion_pro_depth_rel_rgb_py} 0" rpy="0 0 0" />
+      <parent link="door_asus/camera_rgb_frame" />
+      <child link="door_asus/camera_depth_frame" />
+    </joint>
+    <link name="door_asus/camera_depth_frame"/>
+    <joint name="door_asus/camera_depth_optical_joint" type="fixed">
+      <origin xyz="0 0 0" rpy="${-M_PI/2} 0 ${-M_PI/2}" />
+      <parent link="door_asus/camera_depth_frame" />
+      <child link="door_asus/camera_depth_optical_frame" />
+    </joint>
+    <link name="door_asus/camera_depth_optical_frame"/>
+    <!-- Asus mount -->
+    <joint name="door_asus/mount_asus_xtion_pro_joint" type="fixed">
+      <origin xyz="-0.1024 0.0 0.272" rpy="0 0 0"/>
+      <parent link="${parent}"/>
+      <child link="door_asus/mount_asus_xtion_pro_link"/>
+    </joint>
+    <link name="door_asus/mount_asus_xtion_pro_link">
+      <visual>
+        <origin xyz="0 0 0" rpy="${-M_PI/2} 0 0"/>
+        <geometry>
+          <mesh filename="package://turtlebot_description/meshes/sensors/xtion_pro_stack.dae"/>
+        </geometry>
+      </visual>
+      <collision>
+        <origin xyz="0.0 0.0 0.0" rpy="0 0 0" />
+        <geometry>
+        <box size="0.0330 0.2760 0.0120"/>
+      </geometry>
+      </collision>
+      <inertial>
+        <mass value="0.170" />
+        <origin xyz="0 0 0" />
+        <inertia ixx="0.001152600" ixy="0.0" ixz="0.0"
+                 iyy="0.000148934" iyz="0.0"
+                 izz="0.001154654" />
+      </inertial>
+    </link>
   </xacro:macro>
 </robot>

Commit message: door detection working nicely, except maybe half open doors

File: hardware/urdf/sensors/own_sensors.urdf.xacro (robot description, xacro)
@@ -115,6 +115,6 @@
     <!-- Door detection Asus -->
     <joint name="door_asus/camera_joint" type="fixed">
-      <origin xyz="-0.18 -0.03 0.65"
-              rpy="-0.035 -1.13 0.07"/>
+      <origin xyz="-0.25 0.0 0.65"
+              rpy="-0.035 -1.13 0.06"/>
       <parent link="${parent}"/>
       <child link="door_asus/camera_link" />

Commit message: ATTENTION: WITH BUG
some writing
calc move time now with float position
door asus new pose
unvisited rooms good values -> will always be visited
min value now start_value/2 in object map

File: hardware/urdf/sensors/own_sensors.urdf.xacro (robot description, xacro)
@@ -115,6 +115,6 @@
     <!-- Door detection Asus -->
     <joint name="door_asus/camera_joint" type="fixed">
-      <origin xyz="-0.25 0.0 0.65"
-              rpy="-0.035 -1.13 0.06"/>
+      <origin xyz="-0.25 0.0 0.62"
+              rpy="-0.035 -1.2 0.06"/>
       <parent link="${parent}"/>
       <child link="door_asus/camera_link" />

Commit message: explorer: ensure changing goal if former goal is inaccessible fixed handling exploration goal being in robot footprint main ASUS tranformation updated exploration hl planner function updated parameter changes

File: hardware/urdf/sensors/own_sensors.urdf.xacro (robot description, xacro)
@@ -12,6 +12,6 @@
     <!-- Main Asus -->
     <joint name="camera_joint" type="fixed">
-      <origin xyz="-0.18 0.0 0.98"
-              rpy="-0.025 0.17 -0.008"/>
+      <origin xyz="-0.18 0.03 1.02"
+              rpy="-0.02 0.16 -0.008"/>
       <parent link="${parent}"/>
       <child link="camera_link" />
